File: board/enocean-heater-control.kicad_sch (KiCad schematic)
At the start: 4 parts, among them J1 USB_C_Receptacle_PowerOnly_6P, J109 Conn_01x02

Commit message: redo board with STM32G0B0CET
Parts:
- J1: LCSC (none) -> C165948
- J109: LCSC (none) -> C3330556
- R1, R2: LCSC (none) -> C25905
Changed lines of the file:
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@@
+      (effects (font (size 1.27 1.27)) hide)
+    )
+    (property "LCSC" "C165948" (at 39.37 81.28 0)
       (effects (font (size 1.27 1.27)) hide)
     )
@@
       (effects (font (size 1.27 1.27)) hide)
     )
+    (property "LCSC" "C25905" (at 59.69 101.6 0)
+      (effects (font (size 1.27 1.27)) hide)
+    )
     (pin "1")
     (pin "2")
@@
     )
     (property "Datasheet" "~" (at 154.94 109.22 0)
+      (effects (font (size 1.27 1.27)) hide)
+    )
+    (property "LCSC" "C3330556" (at 154.94 109.22 0)
       (effects (font (size 1.27 1.27)) hide)
     )
@@
       (effects (font (size 1.27 1.27)) hide)
     )
+    (property "LCSC" "C25905" (at 57.15 101.6 0)
+      (effects (font (size 1.27 1.27)) hide)
+    )
